File: home-IR-control/IR-controller-board-PCB/board.sch (EAGLE design)
At the start: 7 parts, among them J2 USB-TYPE-C-31-M-12, U1 CH340C

Commit message: PCB update
Parts:
- removed D2: B5819W, angrypig7-Diodes:DIODE-SCHOTTKY_SOD-123
- removed J2: USB-TYPE-C-31-M-12, angrypig7-Connectors:USB-TYPE-C-31-M-12
- added C3, C4, C5, C8: 22uF, angrypig7-RCL:C-NON-POLC0805
- added C6, C7: 100nF, angrypig7-RCL:C-NON-POLC0402
- added D1: B5819W, angrypig7-Diodes:DIODE-SCHOTTKY_SOD-123
- added J1: USB-TYPE-C-31-M-17, angrypig7-Connectors-USB:USB-TYPE-C-31-M-17
- added JP1: (no value), angrypig7-Connectors-PinHeads:PINHD-1X4
- added M1: (no value), angrypig7-Boards:ESP8266-12E
- added R1, R2: 4.7k, angrypig7-RCL:RR0402
- added R5, R6, R7, R8: 10k, angrypig7-RCL:RR0402
- added S1: RST, angrypig7-Switches:SWITCH-SPST-SMD-3.0X4.0MM
- added S2: FLASH, angrypig7-Switches:SWITCH-SPST-SMD-3.0X4.0MM
- C1: LCSC (none) -> C1525
- C2: value 100nF -> 22uF; device angrypig7-RCL:C-NON-POLC0402 -> angrypig7-RCL:C-NON-POLC0805; LCSC C1525 -> C45783
- R3, R4: value 4.7k -> 10k; LCSC C25900 -> (none)
- U1: value CH340C -> AMS1117_SOT223; device angrypig7-IC:CH340C -> angrypig7-IC-Power:AMS1117_SOT223; LCSC (none) -> C6186
Connections:
- removed net N$3: U1.RTS
- removed net N$4: U1.CTS
- removed net USB_N: J2.D-, U1.D-
- removed net USB_P: J2.D+, U1.D+
- new net ESP_ADC: M1.ADC, R8.2
- new net ESP_EN: M1.EN, R4.2
- new net ESP_GPIO0: M1.GPIO0, R5.2, S2.1
- new net ESP_GPIO15: M1.GPIO15, R7.2
- new net ESP_GPIO2: M1.GPIO2, R6.2
- new net ESP_RST: C6.1, M1.RST, R3.2, S1.1
- new net ESP_RST1: C7.1
- new net GND1: C7.2
- net 3V3: now also C3.1, C4.1, C5.1, C8.1, JP1.1, M1.VCC, R3.1, R4.1, R5.1, R6.1, U1.OUT; no longer C1.1, U1.V3, U1.VCC
- net 5V: now also C1.1, D1.C, U1.VIN; no longer D2.C
- net 5V_IN1: now also D1.A, J1.VBUS; no longer D2.A, J2.VBUS
- net GND: now also C3.2, C4.2, C5.2, C6.2, C8.2, J1.GND, J1.SHIELD, JP1.4, M1.GND, R1.1, R2.1, R7.1, R8.1, S1.2, S2.2; no longer J2.GND, J2.SHIELD, R3.1, R4.1
- net N$1: now also J1.CC1, R2.2; no longer J2.CC1, R3.2
- net N$2: now also J1.CC2, R1.2; no longer J2.CC2, R4.2
- net UART_RX: now also JP1.2, M1.RXD; no longer U1.RX
- net UART_TX: now also JP1.3, M1.TXD; no longer U1.TX
Other:
- moved on the sheet: C1, C2, R3, R4
